File: Development/touch_controller/touch_controller.brd (EAGLE design)
At the start: 50 x 50 mm, 44 parts, among them IC1 LPC812M101JDH16, IC2 CY8C201A0-SX2I, IC3 BMA250E, SW1 SK-12D01-VG4, U1 RN4020-V/RM123

Commit message: touch controller rev1
Routing:
- net GND: vias 11 -> 60
- added copper zone on layer 1, net GND
Changed lines of the file:
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@@
 <hole x="15" y="45" drill="3.2"/>
 <rectangle x1="25" y1="32.3" x2="57.9" y2="49.9" layer="42"/>
+<rectangle x1="25" y1="32" x2="58" y2="50" layer="41"/>
+<rectangle x1="34" y1="30" x2="37" y2="32" layer="41"/>
+<rectangle x1="44.5" y1="24.2" x2="45.5" y2="24.3" layer="41"/>
+<rectangle x1="38.1" y1="8.2" x2="38.5" y2="8.3" layer="41"/>
+<rectangle x1="23.9" y1="5.2" x2="24.4" y2="5.3" layer="41"/>
+<rectangle x1="34.1" y1="16.6" x2="34.6" y2="16.8" layer="41"/>
+<rectangle x1="34.2" y1="12.8" x2="34.6" y2="12.9" layer="41"/>
 </plain>
 <attributes>
@@
 <element name="TP8" library="test_pin" package="HT-0720-10" value="HT-0720-10" x="8.7375" y="41.2625"/>
 <element name="TP9" library="test_pin" package="HT-0720-10" value="HT-0720-10" x="25" y="25"/>
-<element name="IC3" library="acceleration_sensor" package="LGA-12" value="BMA250E" x="25" y="28.5"/>
+<element name="IC3" library="acceleration_sensor" package="LGA-12" value="BMA250E" x="25" y="28.5" smashed="yes">
+<attribute name="NAME" x="24.05" y="26.25" size="0.8128" layer="21" font="vector"/>
+</element>
 <element name="C3" library="generic" package="SMD1608_REDUCED" value="" x="27.4" y="28.5" smashed="yes" rot="R90">
 <attribute name="NAME" x="28.85" y="27.9" size="0.8128" layer="25" font="vector" rot="R90"/>
@@
 </element>
 <element name="C4" library="generic" package="SMD1608_REDUCED" value="" x="21.5" y="28.2" smashed="yes" rot="R180">
-<attribute name="NAME" x="23" y="27.85" size="0.8128" layer="25" font="vector"/>
+<attribute name="NAME" x="20.9" y="28.75" size="0.8128" layer="25" font="vector"/>
 <attribute name="VALUE" x="22.3" y="29.85" size="0.8128" layer="27" font="vector" rot="R180"/>
 </element>
@@
 <element name="R10" library="generic" package="SMD1608_REDUCED" value="" x="8.8" y="37.5" rot="R90"/>
 <element name="R11" library="generic" package="SMD1608_REDUCED" value="" x="21.5" y="25.6" smashed="yes">
-<attribute name="NAME" x="20" y="26.05" size="0.8128" layer="25" font="vector" rot="R180"/>
+<attribute name="NAME" x="20.5" y="24.15" size="0.8128" layer="25" font="vector"/>
 <attribute name="VALUE" x="20.7" y="23.95" size="0.8128" layer="27" font="vector"/>
 </element>
@@
 <wire x1="30.4" y1="12.4" x2="30.125" y2="12.675" width="0.3048" layer="1"/>
 <wire x1="30.125" y1="12.675" x2="30.125" y2="13.3" width="0.3048" layer="1"/>
+<polygon width="0.3048" layer="1">
+<vertex x="0" y="0"/>
+<vertex x="50" y="0"/>
+<vertex x="50" y="50"/>
+<vertex x="0" y="50"/>
+</polygon>
+<via x="23" y="48" extent="1-16" drill="0.4"/>
+<via x="19" y="45" extent="1-16" drill="0.4"/>
+<via x="11" y="43" extent="1-16" drill="0.4"/>
+<via x="5" y="37" extent="1-16" drill="0.4"/>
+<via x="15" y="36" extent="1-16" drill="0.4"/>
+<via x="11" y="35" extent="1-16" drill="0.4"/>
+<via x="11" y="31" extent="1-16" drill="0.4"/>
+<via x="2" y="29" extent="1-16" drill="0.4"/>
+<via x="2" y="20" extent="1-16" drill="0.4"/>
+<via x="11" y="20" extent="1-16" drill="0.4"/>
+<via x="11" y="14" extent="1-16" drill="0.4"/>
+<via x="7" y="10" extent="1-16" drill="0.4"/>
+<via x="12" y="5" extent="1-16" drill="0.4"/>
+<via x="18" y="2" extent="1-16" drill="0.4"/>
+<via x="40" y="7" extent="1-16" drill="0.4"/>
+<via x="46" y="14" extent="1-16" drill="0.4"/>
+<via x="39" y="16" extent="1-16" drill="0.4"/>
+<via x="35" y="12" extent="1-16" drill="0.4"/>
+<via x="31" y="12" extent="1-16" drill="0.4"/>
+<via x="28" y="18" extent="1-16" drill="0.4"/>
+<via x="25" y="18" extent="1-16" drill="0.4"/>
+<via x="24" y="17" extent="1-16" drill="0.4"/>
+<via x="35" y="20" extent="1-16" drill="0.4"/>
+<via x="48" y="31" extent="1-16" drill="0.4"/>
+<via x="42" y="31" extent="1-16" drill="0.4"/>
+<via x="38" y="31" extent="1-16" drill="0.4"/>
+<via x="30" y="31" extent="1-16" drill="0.4"/>
+<via x="29" y="26" extent="1-16" drill="0.4"/>
+<via x="14" y="30" extent="1-16" drill="0.4"/>
+<via x="19" y="32" extent="1-16" drill="0.4"/>
+<via x="24" y="35" extent="1-16" drill="0.4"/>
+<via x="23" y="40" extent="1-16" drill="0.4"/>
+<via x="28" y="22" extent="1-16" drill="0.4"/>
+<via x="3" y="26.6" extent="1-16" drill="0.4"/>
+<via x="3" y="22.7" extent="1-16" drill="0.4"/>
+<via x="16.3" y="23.5" extent="1-16" drill="0.4"/>
+<via x="18.1" y="24.9" extent="1-16" drill="0.4"/>
+<via x="15.7" y="20.4" extent="1-16" drill="0.4"/>
+<via x="15.7" y="16.5" extent="1-16" drill="0.4"/>
+<via x="15.7" y="12.6" extent="1-16" drill="0.4"/>
+<via x="22" y="17" extent="1-16" drill="0.4"/>
+<via x="17.4" y="11.4" extent="1-16" drill="0.4"/>
+<via x="9" y="25.6" extent="1-16" drill="0.4"/>
+<via x="8.6" y="29.3" extent="1-16" drill="0.4"/>
+<via x="24.4" y="32.6" extent="1-16" drill="0.4"/>
+<via x="12.3" y="24.2" extent="1-16" drill="0.4"/>
+<via x="44.7" y="18.9" extent="1-16" drill="0.4"/>
+<via x="42.8" y="16.5" extent="1-16" drill="0.4"/>
+<via x="33.9" y="18.3" extent="1-16" drill="0.4"/>
 </signal>
 <signal name="N$1">
