File: Development/touch_controller/touch_controller.sch (EAGLE design)
At the start: 0 parts

Commit message: add library
Parts:
- added BAT1: CH004-2032LF, battery:CH004-2032LF
- added C1, C2, C3, C4, C5, C6: (no value), generic:CAPACITOR1608_REDUCED
- added IC1: LPC812M101JDH16, micro_controller:LPC812M101JDH16
- added IC2: CY8C201A0-SX2I, touch_sensor:CY8C201A0-SX2I
- added IC3: BMA250E, acceleration_sensor:BMA250E
- added JP1: (no value), header:M06NOSILK
- added LED1, LED2, LED3: (no value), generic:LED1608_REDUCED
- added R1, R10, R11, R12, R13, R14, R15, R16, R17, R18, R19, R2, R3, R4, R5, R6, R7, R8, R9: (no value), generic:RESISTOR1608_REDUCED
- added SW1: SK-12D01-VG4, switch:SK-12D01-VG4
- added TP1, TP2, TP3, TP4, TP5, TP6, TP7, TP8, TP9: HT-0720-10, test_pin:HT-0720-10
- added U1: RN4020-V/RM123, com_module:RN4020-V/RM123
Connections:
- new net +3V3: C1.1, C2.1, C3.1, C4.1, C5.1, IC1.VDD, IC2.VDD, IC3.PS, IC3.VDD, IC3.VDDIO, JP1.3, R1.1, R12.1, R17.1, R18.1, R2.1, SW1.P$3, U1.VDD
- new net BLE_RX: IC1.PIO0_7, U1.UART_RX
- new net BLE_TX: IC1.PIO0_6/VDDCMP, U1.UART_TX
- new net CMD/MLDP: IC1.PIO0_9/XTALOUT, R16.1, U1.CMD/MLDP
- new net GND: BAT1.-, C1.2, C2.2, C3.2, C4.2, C5.2, C6.1, IC1.VSS, IC2.VSS, IC3.GND, IC3.GNDIO, IC3.NC, IC3.SDO, JP1.1, LED1.K, LED2.K, LED3.K, R16.2, R19.2, U1.GND@1, U1.GND@2, U1.GND@3, U1.GND@4
- new net GP0_0: IC2.GP0_0, R3.1
- new net GP0_1: IC2.GP0_1, R4.1
- new net GP0_2: IC2.GP0_2, R5.1
- new net GP0_3: IC2.GP0_3, R6.1
- new net GP0_4: IC2.GP0_4, R7.1
- new net GP1_0: IC2.GP1_0, R8.1
- new net GP1_1: IC2.GP1_1, R9.1
- new net GP1_2: IC2.GP1_2, R10.1
- new net GP1_3: IC2.GP1_3, R11.1
- new net GP1_4: IC2.GP1_4
- new net ISP_EN: IC1.PIO0_12, JP1.6
- new net ISP_RXD: IC1.PIO0_0/ACMP_I1/TDO, JP1.4
- new net ISP_TXD: IC1.PIO0_4/WAKEUP/!TRST, JP1.5
- new net N$1: BAT1.+, SW1.P$2
- new net N$10: R10.2, TP8.P$1
- new net N$11: R11.2, TP9.P$1
- new net N$12: R19.1, U1.SPI/!PIO
- new net N$14: LED1.A, R13.2
- new net N$15: LED2.A, R14.2
- new net N$16: LED3.A, R15.2
- new net N$2: C6.2, IC2.CSINT
- new net N$3: R3.2, TP1.P$1
- new net N$4: R4.2, TP2.P$1
- new net N$5: R5.2, TP3.P$1
- new net N$6: R6.2, TP4.P$1
- new net N$7: R7.2, TP5.P$1
- new net N$8: R8.2, TP6.P$1
- new net N$9: R9.2, TP7.P$1
- new net PIO1: R13.1, U1.PIO1/SCK
- new net PIO2: R14.1, U1.MLDP_EV/PIO2/CS
- new net PIO3: R15.1, U1.WS/PIO3/MOSI
- new net RST: IC1.!RESET!/PIO0_5, JP1.2, R12.2
- new net SCL: IC1.PIO0_11, IC2.I2CSCL, IC3.SCX, R1.2
- new net SDA: IC1.PIO0_10, IC2.I2CSDA, IC3.SDX, R2.2
- new net WAKE_HW: IC1.PIO0_8/XTALIN, R18.2, U1.WAKE_HW
- new net WAKE_SW: IC1.PIO0_1/ACMP_I2/CLKIN/TDI, R17.2, U1.WAKE_SW
