File: Development/sphere_robo/sphere_robo.brd (EAGLE design)
At the start: 100 x 80 mm, 0 parts

Commit message: test
Parts:
- added U1: RN4020-V/RM123, com_module:RN4020
Changed lines of the file:
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@@
 </autorouter>
 <elements>
+<element name="U1" library="com_module" package="RN4020" value="RN4020-V/RM123" x="-13.97" y="2.54"/>
 </elements>
 <signals>

Commit message: sphere_robo設計開始
Parts:
- added C1, C2, C3, C4, C5, C6, C7, C8, R1, R13, R14, R15, R2, R3, R4: (no value), generic:SMD1608_REDUCED
- added C10, C9: (no value), generic:PANASONIC_D
- added IC1: ATMEGA328P-AU, AVR:TQFP32-08
- added J1: DM3AT-SF-PEJM5, SDcard:DM3AT-SF-PEJM5
- added JP1: (no value), header:1X06-NOSILK
- added LED1, LED2, LED3: (no value), generic:LED1608_REDUCED
- added R10, R11, R12, R5, R6, R7, R8, R9: 100k, generic:SMD1608_REDUCED
- added U$1: VS1053B, MP3:LQFP48
Connections:
- new net +1V8: U$1.P$24, U$1.P$31, U$1.P$5, U$1.P$7
- new net +3V3: C1.1, C2.1, C4.2, IC1.18, IC1.20, IC1.4, IC1.6, J1.4(VDD), JP1.3, R1.1, R14.1, R15.1, R5.1, U$1.P$14, U$1.P$19, U$1.P$32, U$1.P$38, U$1.P$43, U$1.P$45, U$1.P$6
- new net AGND: U$1.P$37, U$1.P$40, U$1.P$41, U$1.P$47
- new net BLE_RX: IC1.28, U1.6
- new net BLE_TX: IC1.27, U1.5
- new net CMD/MLDP: IC1.25, U1.8
- new net GBUF: R11.1, U$1.P$42
- new net GND: C1.2, C2.2, C4.1, C5.2, C6.2, C7.2, C8.2, IC1.21, IC1.3, IC1.5, J1.6(GND), J1.SHIELD@1, J1.SHIELD@2, J1.SHIELD@3, J1.SHIELD@4, JP1.1, LED1.K, LED2.K, LED3.K, R10.2, R13.2, R6.2, R7.2, R8.2, R9.2, U$1.P$10, U$1.P$11, U$1.P$12, U$1.P$16, U$1.P$20, U$1.P$21, U$1.P$22, U$1.P$35, U$1.P$4, U$1.P$9, U1.1, U1.16, U1.24, U1.9
- new net MISO: IC1.16, J1.7(DAT0), U$1.P$30
- new net MOSI: IC1.15, J1.3(CMD), U$1.P$29
- new net MP3-CS: IC1.10, U$1.P$23
- new net MP3-DCS: IC1.11, U$1.P$13
- new net MP3-DREQ: IC1.32, U$1.P$8
- new net MP3-RST: IC1.12, R10.1, U$1.P$3
- new net N$1: C3.2, IC1.29, R1.2
- new net N$10: C5.1, U$1.P$44
- new net N$11: R13.1, U1.17
- new net N$12: R5.2, U$1.P$26
- new net N$13: U$1.P$46
- new net N$15: C7.1, R12.1, U$1.P$18
- new net N$17: C6.1, R11.2
- new net N$19: C8.1, R12.2, U$1.P$17
- new net N$2: C3.1, JP1.6
- new net N$3: LED1.A, R2.2
- new net N$4: LED2.A, R3.2
- new net N$5: LED3.A, R4.2
- new net N$6: R6.1, U$1.P$25
- new net N$7: R7.1, U$1.P$36
- new net N$8: R8.1, U$1.P$34
- new net N$9: R9.1, U$1.P$33
- new net PIO1: R2.1, U1.10
- new net PIO2: R3.1, U1.11
- new net PIO3: R4.1, U1.12
- new net RXD: IC1.30, JP1.4
- new net SCK: IC1.17, J1.5(CLK), U$1.P$28
- new net SD-CS: IC1.13, J1.2(CD/DAT3)
- new net TXD: IC1.31, JP1.5
- new net WAKE_HW: IC1.24, R15.2, U1.15
- new net WAKE_SW: IC1.23, R14.2, U1.7
